Commit message: done with basic gazebo simulation

File: description/robot.urdf.xacro (robot description, xacro)
@@ -1,5 +1,5 @@
 <?xml version="1.0"?>
 <robot xmlns:xacro="http://www.ros.org/wiki/xacro"  name="robot">
-    <!-- Example link -->
     <xacro:include filename="robot_core.xacro"/>
+    <xacro:include filename="gazebo_control.xacro"/>
 </robot>

File: description/robot_core.xacro (robot description, xacro)
@@ -1,5 +1,5 @@
 <?xml version="1.0"?>
 <robot xmlns:xacro="http://www.ros.org/wiki/xacro">
-    <xacro:include filename="inertial_macros.xacro"/>
+    <xacro:include filename="$(find my_bot)/description/inertial_macros.xacro"/>
     <material name="white">
         <color rgba="1 1 1 1" />
@@ -72,5 +72,5 @@
                 <cylinder radius="0.5" length="0.2"/>
             </geometry>
-            <material name="transparent_gray"/>
+            <material name="cyan"/>
         </collision>
         <xacro:inertial_cylinder mass="5" length="0.2" radius="0.5">
@@ -78,4 +78,7 @@
         </xacro:inertial_cylinder>
     </link>
+    <gazebo reference="chassis_link">
+        <material>Gazebo/cWhite</material>
+    </gazebo>
     <!-- left wheel link-->
     <joint name="left_wheel_joint" type="continuous">
@@ -102,4 +105,7 @@
         </xacro:inertial_cylinder>
     </link>
+    <gazebo reference="left_wheel_link">
+        <material>Gazebo/Black</material>
+    </gazebo>
     <!-- right wheel link-->
     <joint name="right_wheel_joint" type="continuous">
@@ -107,5 +113,5 @@
         <child link="right_wheel_link"/>
         <origin xyz="0 -0.5 0" rpy="${pi/2} 0 0"/>
-        <axis xyz="0 0 -1"/>
+        <axis xyz="0 0 1"/>
     </joint>
     <link name="right_wheel_link">
@@ -126,4 +132,7 @@
         </xacro:inertial_cylinder>
     </link>
+    <gazebo reference="right_wheel_link">
+        <material>Gazebo/Black</material>
+    </gazebo>
     <!--caster wheel limk-->
     <joint name="back_caster_wheel_joint" type="fixed">
@@ -149,4 +158,7 @@
         </xacro:inertial_sphere>
     </link>
+    <gazebo reference="back_caster_wheel_link">
+        <material>Gazebo/Black</material>
+    </gazebo>
     <joint name="front_caster_wheel_joint" type="fixed">
         <parent link="base_link"/>
@@ -171,3 +183,14 @@
         </xacro:inertial_sphere>
     </link>
+    <gazebo reference="front_caster_wheel_link">
+        <material>Gazebo/Black</material>
+    </gazebo>
+    <gazebo reference="front_caster_wheel_link">
+        <mu1>0.01</mu1>
+        <mu2>0.01</mu2>
+    </gazebo>
+    <gazebo reference="back_caster_wheel_link">
+        <mu1>0.01</mu1>
+        <mu2>0.01</mu2>
+    </gazebo>
 </robot>
