Commit message: done with lidar

File: description/gazebo_control.xacro (robot description, xacro)
@@ -2,5 +2,10 @@
 <robot xmlns:xacro="http://www.ros.org/wiki/xacro"  name="robot">
     <gazebo>
-        <plugin name="diff_drive_controller" filename="libgazebo_ros_diff_drive.so">
+        <plugin name="diff_drive" filename="libgazebo_ros_diff_drive.so">
+            <ros>
+                <namespace>/</namespace>
+                <remapping>cmd_vel:=cmd_vel</remapping>
+                <remapping>odom:=odom</remapping>
+            </ros>
             <!--Wheel information-->
             <left_joint>left_wheel_joint</left_joint>
@@ -14,7 +19,10 @@
             <odometry_frame>odom</odometry_frame>
             <robot_base_frame>base_link</robot_base_frame>
+            <command_topic>cmd_vel</command_topic>
+            <odometry_topic>odom</odometry_topic>
             <publish_odom>true</publish_odom>
             <publish_odom_tf>true</publish_odom_tf>
             <publish_wheel_tf>true</publish_wheel_tf>
+             <update_rate>50</update_rate>
         </plugin>
     </gazebo>

File: description/robot.urdf.xacro (robot description, xacro)
@@ -3,3 +3,4 @@
     <xacro:include filename="robot_core.xacro"/>
     <xacro:include filename="gazebo_control.xacro"/>
+    <xacro:include filename="lidar.xacro"/>
 </robot>

File: description/robot_core.xacro (robot description, xacro)
@@ -79,5 +79,5 @@
     </link>
     <gazebo reference="chassis_link">
-        <material>Gazebo/cWhite</material>
+        <material>Gazebo/White</material>
     </gazebo>
     <!-- left wheel link-->
@@ -108,4 +108,12 @@
         <material>Gazebo/Black</material>
     </gazebo>
+    <gazebo reference="left_wheel_link">
+        <mu1>1.0</mu1>
+        <mu2>1.0</mu2>
+    </gazebo>
+    <gazebo reference="right_wheel_link">
+        <mu1>1.0</mu1>
+        <mu2>1.0</mu2>
+    </gazebo>
     <!-- right wheel link-->
     <joint name="right_wheel_joint" type="continuous">
